File: smartlight/smartlight.kicad_sch (KiCad schematic)
At the start: 16 parts, among them J1 Conn_01x06, J2 Conn_01x05, SW1 RESET, SW2 IO0, U1 ESP-12F

Commit message: update
Parts:
- removed SW1: RESET, Button_Switch_SMD:SW_Push_SPST_NO_Alps_SKRK, symbol Switch:SW_Push
- removed SW2: IO0, Button_Switch_SMD:SW_Push_SPST_NO_Alps_SKRK, symbol Switch:SW_Push
- J2: footprint Connector_PinHeader_1.27mm:PinHeader_1x05_P1.27mm_Vertical -> taki-library:ENDO_CONTROLLER
- R1, R2, R3, R4, R5, R6, R7, R8: footprint Resistor_SMD:R_0603_1608Metric -> Resistor_SMD:R_0402_1005Metric

Commit message: before swapping pin snapshot
Parts:
- removed D1: LED, LED_SMD:LED_0603_1608Metric, symbol Device:LED
- removed R8: 2k, Resistor_SMD:R_0402_1005Metric, symbol Device:R_Small
- added FID1, FID2, FID3, FID4: Fiducial, Fiducial:Fiducial_1mm_Mask2mm, symbol Mechanical:Fiducial
- added H1, H2, H3, H4: mousebite, taki-library:mousebites_1mm, symbol Mechanical:MountingHole
Connections:
- no-connect marks 11 -> 12

Commit message: コントローラー管制
Connections:
- net +3V3: now also J2.2 (Pin_2); no longer J2.4 (Pin_4)
- net at R2.2: now also J2.5 (Pin_5); no longer J2.1 (Pin_1)
- net at R1.2: now also J2.4 (Pin_4); no longer J2.2 (Pin_2)
Other:
- moved on the sheet: FID1, FID2, FID3, FID4, H1, H2, H3, H4, J2
Changed lines of the file:
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@@
 	)
 	(no_connect
-		(at 215.9 87.63)
+		(at 214.63 87.63)
 	)
 	(no_connect
@@
 	(wire
 		(pts
-			(xy 215.9 82.55) (xy 212.09 82.55)
+			(xy 214.63 82.55) (xy 212.09 82.55)
 		)
 		(stroke
@@
 	(wire
 		(pts
-			(xy 215.9 77.47) (xy 199.39 77.47)
+			(xy 214.63 77.47) (xy 199.39 77.47)
 		)
 		(stroke
@@
 	(wire
 		(pts
-			(xy 208.28 85.09) (xy 215.9 85.09)
+			(xy 208.28 85.09) (xy 214.63 85.09)
 		)
 		(stroke
@@
 	(wire
 		(pts
-			(xy 199.39 80.01) (xy 215.9 80.01)
+			(xy 199.39 80.01) (xy 214.63 80.01)
 		)
 		(stroke
@@
 	(symbol
 		(lib_id "Mechanical:Fiducial")
-		(at 238.76 144.78 0)
+		(at 241.3 149.86 0)
 		(unit 1)
 		(exclude_from_sim yes)
@@
 		(fields_autoplaced yes)
 		(property "Reference" "FID2"
-			(at 241.3 143.5099 0)
+			(at 243.84 148.5899 0)
 			(effects
 				(font
@@
 		)
 		(property "Value" "Fiducial"
-			(at 241.3 146.0499 0)
+			(at 243.84 151.1299 0)
 			(effects
 				(font
@@
 		)
 		(property "Footprint" "Fiducial:Fiducial_1mm_Mask2mm"
-			(at 238.76 144.78 0)
+			(at 241.3 149.86 0)
 			(effects
 				(font
@@
 		)
 		(property "Datasheet" "~"
-			(at 238.76 144.78 0)
+			(at 241.3 149.86 0)
 			(effects
 				(font
@@
 		)
 		(property "Description" "Fiducial Marker"
-			(at 238.76 144.78 0)
+			(at 241.3 149.86 0)
 			(effects
 				(font
@@
 	(symbol
 		(lib_id "Mechanical:MountingHole")
-		(at 36.83 119.38 0)
+		(at 209.55 151.13 0)
 		(unit 1)
 		(exclude_from_sim yes)
@@
 		(fields_autoplaced yes)
 		(property "Reference" "H3"
-			(at 39.37 118.1099 0)
+			(at 212.09 149.8599 0)
 			(effects
 				(font
@@
 		)
 		(property "Value" "mousebite"
-			(at 39.37 120.6499 0)
+			(at 212.09 152.3999 0)
 			(effects
 				(font
@@
 		)
 		(property "Footprint" "taki-library:mousebites_1mm"
-			(at 36.83 119.38 0)
+			(at 209.55 151.13 0)
 			(effects
 				(font
@@
 		)
 		(property "Datasheet" "~"
-			(at 36.83 119.38 0)
+			(at 209.55 151.13 0)
 			(effects
 				(font
@@
 		)
 		(property "Description" "Mounting Hole without connection"
-			(at 36.83 119.38 0)
+			(at 209.55 151.13 0)
 			(effects
 				(font
@@
 	(symbol
 		(lib_id "Mechanical:MountingHole")
-		(at 36.83 113.03 0)
+		(at 191.77 157.48 0)
 		(unit 1)
 		(exclude_from_sim yes)
@@
 		(fields_autoplaced yes)
 		(property "Reference" "H2"
-			(at 39.37 111.7599 0)
+			(at 194.31 156.2099 0)
 			(effects
 				(font
@@
 		)
 		(property "Value" "mousebite"
-			(at 39.37 114.2999 0)
+			(at 194.31 158.7499 0)
 			(effects
 				(font
@@
 		)
 		(property "Footprint" "taki-library:mousebites_1mm"
-			(at 36.83 113.03 0)
+			(at 191.77 157.48 0)
 			(effects
 				(font
@@
 		)
 		(property "Datasheet" "~"
-			(at 36.83 113.03 0)
+			(at 191.77 157.48 0)
 			(effects
 				(font
@@
 		)
 		(property "Description" "Mounting Hole without connection"
-			(at 36.83 113.03 0)
+			(at 191.77 157.48 0)
 			(effects
 				(font
@@
 	(symbol
 		(lib_id "Mechanical:Fiducial")
-		(at 223.52 152.4 0)
+		(at 226.06 157.48 0)
 		(unit 1)
 		(exclude_from_sim yes)
@@
 		(fields_autoplaced yes)
 		(property "Reference" "FID3"
-			(at 226.06 151.1299 0)
+			(at 228.6 156.2099 0)
 			(effects
 				(font
@@
 		)
 		(property "Value" "Fiducial"
-			(at 226.06 153.6699 0)
+			(at 228.6 158.7499 0)
 			(effects
 				(font
@@
 		)
 		(property "Footprint" "Fiducial:Fiducial_1mm_Mask2mm"
-			(at 223.52 152.4 0)
+			(at 226.06 157.48 0)
 			(effects
 				(font
@@
 		)
 		(property "Datasheet" "~"
-			(at 223.52 152.4 0)
+			(at 226.06 157.48 0)
 			(effects
 				(font
@@
 		)
 		(property "Description" "Fiducial Marker"
-			(at 223.52 152.4 0)
+			(at 226.06 157.48 0)
 			(effects
 				(font
@@
 	(symbol
 		(lib_id "Mechanical:MountingHole")
-		(at 36.83 125.73 0)
+		(at 209.55 157.48 0)
 		(unit 1)
 		(exclude_from_sim yes)
@@
 		(fields_autoplaced yes)
 		(property "Reference" "H4"
-			(at 39.37 124.4599 0)
+			(at 212.09 156.2099 0)
 			(effects
 				(font
@@
 		)
 		(property "Value" "mousebite"
-			(at 39.37 126.9999 0)
+			(at 212.09 158.7499 0)
 			(effects
 				(font
@@
 		)
 		(property "Footprint" "taki-library:mousebites_1mm"
-			(at 36.83 125.73 0)
+			(at 209.55 157.48 0)
 			(effects
 				(font
@@
 		)
 		(property "Datasheet" "~"
-			(at 36.83 125.73 0)
+			(at 209.55 157.48 0)
 			(effects
 				(font
@@
 		)
 		(property "Description" "Mounting Hole without connection"
-			(at 36.83 125.73 0)
+			(at 209.55 157.48 0)
 			(effects
 				(font
@@
 	(symbol
 		(lib_id "Mechanical:MountingHole")
-		(at 36.83 106.68 0)
+		(at 191.77 151.13 0)
 		(unit 1)
 		(exclude_from_sim yes)
@@
 		(fields_autoplaced yes)
 		(property "Reference" "H1"
-			(at 39.37 105.4099 0)
+			(at 194.31 149.8599 0)
 			(effects
 				(font
@@
 		)
 		(property "Value" "mousebite"
-			(at 39.37 107.9499 0)
+			(at 194.31 152.3999 0)
 			(effects
 				(font
@@
 		)
 		(property "Footprint" "taki-library:mousebites_1mm"
-			(at 36.83 106.68 0)
+			(at 191.77 151.13 0)
 			(effects
 				(font
@@
 		)
 		(property "Datasheet" "~"
-			(at 36.83 106.68 0)
+			(at 191.77 151.13 0)
 			(effects
 				(font
@@
 		)
 		(property "Description" "Mounting Hole without connection"
-			(at 36.83 106.68 0)
+			(at 191.77 151.13 0)
 			(effects
 				(font
@@
 	(symbol
 		(lib_id "Mechanical:Fiducial")
-		(at 223.52 144.78 0)
+		(at 226.06 149.86 0)
 		(unit 1)
 		(exclude_from_sim yes)
@@
 		(fields_autoplaced yes)
 		(property "Reference" "FID1"
-			(at 226.06 143.5099 0)
+			(at 228.6 148.5899 0)
 			(effects
 				(font
@@
 		)
 		(property "Value" "Fiducial"
-			(at 226.06 146.0499 0)
+			(at 228.6 151.1299 0)
 			(effects
 				(font
@@
 		)
 		(property "Footprint" "Fiducial:Fiducial_1mm_Mask2mm"
-			(at 223.52 144.78 0)
+			(at 226.06 149.86 0)
 			(effects
 				(font
@@
 		)
 		(property "Datasheet" "~"
-			(at 223.52 144.78 0)
+			(at 226.06 149.86 0)
 			(effects
 				(font
@@
 		)
 		(property "Description" "Fiducial Marker"
-			(at 223.52 144.78 0)
+			(at 226.06 149.86 0)
 			(effects
 				(font
@@
 	(symbol
 		(lib_id "Mechanical:Fiducial")
-		(at 238.76 152.4 0)
+		(at 241.3 157.48 0)
 		(unit 1)
 		(exclude_from_sim yes)
@@
 		(fields_autoplaced yes)
 		(property "Reference" "FID4"
-			(at 241.3 151.1299 0)
+			(at 243.84 156.2099 0)
 			(effects
 				(font
@@
 		)
 		(property "Value" "Fiducial"
-			(at 241.3 153.6699 0)
+			(at 243.84 158.7499 0)
 			(effects
 				(font
@@
 		)
 		(property "Footprint" "Fiducial:Fiducial_1mm_Mask2mm"
-			(at 238.76 152.4 0)
+			(at 241.3 157.48 0)
 			(effects
 				(font
@@
 		)
 		(property "Datasheet" "~"
-			(at 238.76 152.4 0)
+			(at 241.3 157.48 0)
 			(effects
 				(font
@@
 		)
 		(property "Description" "Fiducial Marker"
-			(at 238.76 152.4 0)
+			(at 241.3 157.48 0)
 			(effects
 				(font
@@
 	(symbol
 		(lib_id "Connector_Generic:Conn_01x05")
-		(at 220.98 82.55 0)
+		(at 219.71 82.55 0)
+		(mirror x)
 		(unit 1)
 		(exclude_from_sim no)
@@
 		(on_board yes)
 		(dnp no)
-		(fields_autoplaced yes)
 		(property "Reference" "J2"
-			(at 223.52 81.2799 0)
+			(at 222.25 83.8201 0)
 			(effects
 				(font
@@
 		)
 		(property "Value" "Conn_01x05"
-			(at 223.52 83.8199 0)
+			(at 222.25 81.2801 0)
 			(effects
 				(font
@@
 		)
 		(property "Footprint" "taki-library:ENDO_CONTROLLER"
-			(at 220.98 82.55 0)
+			(at 219.71 82.55 0)
 			(effects
 				(font
@@
 		)
 		(property "Datasheet" "~"
-			(at 220.98 82.55 0)
+			(at 219.71 82.55 0)
 			(effects
 				(font
@@
 		)
 		(property "Description" "Generic connector, single row, 01x05, script generated (kicad-library-utils/schlib/autogen/connector/)"
-			(at 220.98 82.55 0)
-			(effects
-				(font
+			(at 219.71 82.55 0)
+			(effects
+				(font
