File: smartlight/smartlight.kicad_pcb (KiCad board)
At the start: 2 copper layers, 19 x 24.5 mm, 18 parts, among them J1 Conn_01x06, J2 Conn_01x05, SW1 RESET, SW2 IO0, U1 ESP-12F

Commit message: update
Parts:
- removed the REF** at (118.8, 41.0)
- removed SW1: RESET, Button_Switch_SMD:SW_Push_SPST_NO_Alps_SKRK
- removed SW2: IO0, Button_Switch_SMD:SW_Push_SPST_NO_Alps_SKRK
- added REF**: mousebites_1mm, taki-library:mousebites_1mm, F.Cu at (79.5, 50.0)
- added REF**: Fiducial_1mm_Mask2mm, Fiducial:Fiducial_1mm_Mask2mm, F.Cu at (73.5, 70.0)
- added REF**: mousebites_1mm, taki-library:mousebites_1mm, F.Cu at (79.5, 62.5)
- added REF**: Fiducial_1mm_Mask2mm, Fiducial:Fiducial_1mm_Mask2mm, F.Cu at (73.5, 42.5)
- added REF**: Fiducial_1mm_Mask2mm, Fiducial:Fiducial_1mm_Mask2mm, F.Cu at (106.5, 70.0)
- added REF**: mousebites_1mm, taki-library:mousebites_1mm, F.Cu at (100.5, 62.5)
- added REF**: Fiducial_1mm_Mask2mm, Fiducial:Fiducial_1mm_Mask2mm, F.Cu at (106.5, 42.5)
- R8: value 2.1k -> 2k
- turned REF** to 90 degrees
Other:
- board size 19 x 24.5 mm -> 43 x 37.5 mm
- board text added: "↑fiducials"

Commit message: before swapping pin snapshot
Parts:
- removed D1: LED, LED_SMD:LED_0603_1608Metric
- removed R8: 2k, Resistor_SMD:R_0402_1005Metric
- removed REF** (x4): mousebites_1mm, taki-library:mousebites_1mm
- removed REF** (x4): Fiducial_1mm_Mask2mm, Fiducial:Fiducial_1mm_Mask2mm
- added FID1: Fiducial, Fiducial:Fiducial_1mm_Mask2mm, F.Cu at (73.0, 42.0)
- added FID2: Fiducial, Fiducial:Fiducial_1mm_Mask2mm, F.Cu at (107.0, 42.0)
- added FID3: Fiducial, Fiducial:Fiducial_1mm_Mask2mm, F.Cu at (73.0, 70.0)
- added FID4: Fiducial, Fiducial:Fiducial_1mm_Mask2mm, F.Cu at (107.0, 70.0)
- added H1: mousebite, taki-library:mousebites_1mm, F.Cu at (79.5, 62.5)
- added H2: mousebite, taki-library:mousebites_1mm, F.Cu at (79.5, 50.0)
- added H3: mousebite, taki-library:mousebites_1mm, F.Cu at (100.5, 50.0)
- added H4: mousebite, taki-library:mousebites_1mm, F.Cu at (100.5, 62.5)
- moved R2 7.64 mm to (88.8, 65.7)
- moved R1 7.43 mm to (86.2, 66.2), turned to 0 degrees
- moved R5 6.25 mm to (85.2, 65.0)
- moved C2 1.98 mm to (85.7, 67.6)
- moved R6 1.75 mm to (85.2, 63.8)
- moved J2 1.50 mm to (91.0, 71.5)
- moved R3 0.25 mm to (98.0, 67.0)
- moved R4 0.25 mm to (81.5, 66.8)
- moved R7 0.25 mm to (94.0, 67.0)
Connections:
- U1 pad 20: Net-(U1-GPIO5) -> unconnected-(U1-GPIO5-Pad20)
Routing:
- net GND: track 0.00 -> 55.3 mm, vias 0 -> 82
- net +3V3: track 0.00 -> 35.9 mm, vias 0 -> 2
- net RESET: track 0.00 -> 35.1 mm, vias 0 -> 1
- net Net-(U1-EN): track 0.00 -> 22.1 mm, vias 0 -> 2
- net ESP12F_TX: track 0.00 -> 21.5 mm, vias 0 -> 1
- net PWM: track 0.00 -> 20.4 mm, vias 0 -> 2
- net ESP12F_RX: track 0.00 -> 19.8 mm, vias 0 -> 1
- net Net-(U1-GPIO2): track 0.00 -> 18.2 mm, vias 0 -> 2
- net IO0: track 0.00 -> 18.0 mm, vias 0 -> 1
- net Net-(U1-GPIO15): track 0.00 -> 16.8 mm, vias 0 -> 2
- net ON/OFF: track 0.00 -> 15.9 mm, vias 0 -> 2
- net Net-(J2-Pin_2): track 0.00 -> 15.7 mm, vias 0 -> 2
- net Net-(J2-Pin_1): track 0.00 -> 14.2 mm, vias 0 -> 2
- added copper zone on B.Cu, net GND
- added copper zone on F.Cu, net GND
Other:
- board size 43 x 37.5 mm -> 43 x 36 mm

Commit message: コントローラー管制
Connections:
- J2 pad 1: Net-(J2-Pin_1) -> unconnected-(J2-Pin_1-Pad1)
- J2 pad 2: Net-(J2-Pin_2) -> +3V3
- J2 pad 4: +3V3 -> Net-(J2-Pin_4)
- J2 pad 5: unconnected-(J2-Pin_5-Pad5) -> Net-(J2-Pin_5)
- R1 pad 2: Net-(J2-Pin_2) -> Net-(J2-Pin_4)
- R2 pad 2: Net-(J2-Pin_1) -> Net-(J2-Pin_5)
Routing:
- net Net-(J2-Pin_2): track 15.7 -> 0.00 mm, vias 2 -> 0
- net Net-(J2-Pin_1): track 14.2 -> 0.00 mm, vias 2 -> 0
- net Net-(J2-Pin_5): track 0.00 -> 13.8 mm, vias 0 -> 2
- net Net-(J2-Pin_4): track 0.00 -> 10.1 mm, vias 0 -> 2
- net +3V3: track 35.9 -> 40.8 mm
- net GND: track 55.3 -> 52.5 mm, vias 82 -> 88
- net unconnected-(J2-Pin_1-Pad1): track 0.00 -> 2.60 mm

Commit message: update
Parts:
- moved R1 0.15 mm to (86.2, 66.1)
Changed lines of the file:
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@@
 		(tags "capacitor")
 		(property "Reference" "C2"
-			(at 2.5 0 360)
+			(at 2.5 0 0)
 			(layer "F.SilkS")
 			(effects
@@
 		)
 		(property "Value" "1u"
-			(at 0 1.43 360)
+			(at 0 1.43 0)
 			(layer "F.Fab")
 			(effects
@@
 		)
 		(fp_text user "${REFERENCE}"
-			(at 0 0 360)
+			(at 0 0 0)
 			(layer "F.Fab")
 			(effects
@@
 	(footprint "Resistor_SMD:R_0402_1005Metric"
 		(layer "F.Cu")
-		(at 86.25 66.25)
+		(at 86.25 66.1)
 		(descr "Resistor SMD 0402 (1005 Metric), square (rectangular) end terminal, IPC_7351 nominal, (Body size source: IPC-SM-782 page 72, https://www.pcb-3d.com/wordpress/wp-content/uploads/ipc-sm-782a_amendment_1_and_2.pdf), generated with kicad-footprint-generator")
 		(tags "resistor")
 		(property "Reference" "R1"
-			(at -1.95 0 360)
+			(at -1.95 0 0)
 			(layer "F.SilkS")
 			(effects
@@
 		)
 		(property "Value" "100"
-			(at 0 1.17 360)
+			(at 0 1.17 0)
 			(layer "F.Fab")
 			(effects
@@
 		)
 		(fp_text user "${REFERENCE}"
-			(at 0 0 360)
-			(layer "F.Fab")
-			(effects
+			(at 0 0 0)
+			(layer "F.Fab")
+			(effects
